Commit message: urdf updates

File: assets/urdf/ur5/ur5_with_succ.urdf (robot description, URDF)
Before this commit: robot ur5_with_measurement_tool, 11 links, 10 joints
Links:
- link succ_tool: geometry collision mesh filename=meshes/collision/grasped.obj; visual mesh filename=meshes/visual/grasped.obj
