Commit message: taller camera, new bin

File: assets/urdf/custom/cardboardbin.urdf (robot description, URDF)
Before this commit: robot tray, 1 links, 0 joints
Links:
- link tray_base_link: geometry collision mesh filename=meshes/zk_bin.obj scale=1 1 1; visual mesh filename=meshes/zk_bin.obj scale=1 1 1

Commit message: ortho graphic modification

File: assets/urdf/custom/cardboardbin.urdf (robot description, URDF)
Before this commit: robot tray, 1 links, 0 joints
Links:
- link tray_base_link: geometry collision mesh filename=meshes/realbin.obj scale=1 1 1; visual mesh filename=meshes/realbin.obj scale=1 1 1
